File: hardware/pcb/Phishy_WLED/ws28xx_LEDs.kicad_sch (KiCad schematic)
At the start: 16 parts, among them Q1 2N7002L, Q13 BSS138, Q14 BSS138, Q17 BSS138, Q18 BSS138

Commit message: footprints added !
all the footprints are here
Parts:
- R3, R5: footprint (none) -> Resistor_SMD:R_0603_1608Metric
Changed lines of the file:
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@@
       (effects (font (size 1.27 1.27)) (justify right))
     )
-    (property "Footprint" "" (at 161.798 93.98 90)
+    (property "Footprint" "Resistor_SMD:R_0603_1608Metric" (at 161.798 93.98 90)
       (effects (font (size 1.27 1.27)) hide)
     )
@@
       (effects (font (size 1.27 1.27)) (justify right))
     )
-    (property "Footprint" "" (at 80.518 92.71 90)
+    (property "Footprint" "Resistor_SMD:R_0603_1608Metric" (at 80.518 92.71 90)
       (effects (font (size 1.27 1.27)) hide)
     )
@@
       (effects (font (size 1.27 1.27)) (justify right))
     )
-    (property "Footprint" "" (at 80.518 50.8 90)
+    (property "Footprint" "Resistor_SMD:R_0603_1608Metric" (at 80.518 50.8 90)
       (effects (font (size 1.27 1.27)) hide)
     )
@@
       (effects (font (size 1.27 1.27)))
     )
-    (property "Footprint" "" (at 63.5 65.278 90)
+    (property "Footprint" "Resistor_SMD:R_0603_1608Metric" (at 63.5 65.278 90)
       (effects (font (size 1.27 1.27)) hide)
     )
@@
       (effects (font (size 1.27 1.27)) (justify right))
     )
-    (property "Footprint" "" (at 161.798 52.07 90)
+    (property "Footprint" "Resistor_SMD:R_0603_1608Metric" (at 161.798 52.07 90)
       (effects (font (size 1.27 1.27)) hide)
     )
@@
       (effects (font (size 1.27 1.27)))
     )
-    (property "Footprint" "" (at 144.78 66.548 90)
+    (property "Footprint" "Resistor_SMD:R_0603_1608Metric" (at 144.78 66.548 90)
       (effects (font (size 1.27 1.27)) hide)
     )
@@
       (effects (font (size 1.27 1.27)))
     )
-    (property "Footprint" "" (at 144.78 108.458 90)
+    (property "Footprint" "Resistor_SMD:R_0603_1608Metric" (at 144.78 108.458 90)
       (effects (font (size 1.27 1.27)) hide)
     )
@@
       (effects (font (size 1.27 1.27)))
     )
-    (property "Footprint" "" (at 63.5 107.188 90)
-      (effects (font (size 1.27 1.27)) hide)
-    )
+    (property "Footprint" "Resistor_SMD:R_0603_1608Metric" (at 63.5 107.188 90)
+      (effects (font (size 1.27 1.27)) hide)
+    )
